File: hog_power.sch (KiCad schematic (older format))
At the start: 8 parts, among them Q1 Q_PMOS_DGS

Commit message: update
Parts:
- added JP?: Jumper_NO_Small, symbol Jumper_NO_Small
Connections:
- net +5V: now also JP?.2
- net at D1.1 (K), R1.1, U?.3 (VI): now also JP?.1
Other:
- note added: "-- D1,D2: Schottky diodes w/ voltage drop = 0.2 Volts"
- note added: "-- If no need for switching regulator (e.g. no need for 5V on batt power),\ncan use jumper to connect VBATT input to 3.3V LDO directly"
- note added: "-- When VBATT >= 6.6V, op-amp comparator (via op-amp comparator)\n selects VBATT instead of VBUS as input to 3.3V LDO"
- note added: "USB Input (5V)"
- note removed: "D1,D2: Schottky diodes w/ voltage drop = 0.2 Volts"
- note removed: "USB Input"
- moved on the sheet: D1, D2, Q1, R1, R2, U?, U?A
