File: hog32a.kicad_pcb (KiCad board)
At the start: 2 copper layers, 51.6 x 75.9 mm, 39 parts, among them J1 REG:3V3, J10 Conn_01x07, J11 Conn_01x16, J12 dht22, J13 9602-a, J14 satx, J15 Conn_01x05, J16 LBO, J19 9602-b, J2 prog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

Commit message: update
Parts:
- removed J8: Conn_01x01, SMD_Packages:1Pin
Other:
- board text added: "HOG-A-LOG"
- board text added: "http://edgecollective.io/hog-a-log"
- board text removed: "HOGALOG"
- board text removed: "http://edgecollective.io/hogalog"
Changed lines of the file:
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@@
 (kicad_pcb (version 4) (host pcbnew 4.0.7-e2-6376~58~ubuntu16.04.1)
   (general
-    (links 129)
+    (links 128)
     (no_connects 0)
     (area 72.924599 30.404999 124.636601 106.501001)
@@
     (tracks 783)
     (zones 0)
-    (modules 39)
+    (modules 38)
     (nets 46)
   )
@@
     )
   )
-  (module SMD_Packages:1Pin (layer F.Cu)
-    (at 107.0864 45.6692)
-    (descr "module 1 pin (ou trou mecanique de percage)")
-    (tags DEV)
-    (fp_text reference J8 (at 0 -3.50012) (layer F.SilkS)
-      (effects (font (size 1 1) (thickness 0.15)))
-    )
-    (fp_text value Conn_01x01 (at 0.24892 3.74904) (layer F.Fab)
-      (effects (font (size 1 1) (thickness 0.15)))
-    )
-    (fp_line (start -2.49936 -2.49936) (end 2.49936 -2.49936) (layer F.SilkS) (width 0.15))
-    (fp_line (start 2.49936 -2.49936) (end 2.49936 2.49936) (layer F.SilkS) (width 0.15))
-    (fp_line (start 2.49936 2.49936) (end -2.49936 2.49936) (layer F.SilkS) (width 0.15))
-    (fp_line (start -2.49936 2.49936) (end -2.49936 -2.49936) (layer F.SilkS) (width 0.15))
-    (pad 1 smd rect (at 0 0) (size 4.064 4.064) (layers B.Cu F.Paste F.Mask)
-      (net 3 GND))
-  )
   (module Pin_Headers:Pin_Header_Straight_1x07_Pitch2.54mm (layer F.Cu)
     (at 75.0189 32.6898 90)
@@
     (effects (font (size 0.8 0.8) (thickness 0.125)))
   )
-  (gr_text http://edgecollective.io/hogalog (at 97.0788 44.0182) (layer B.SilkS)
+  (gr_text http://edgecollective.io/hog-a-log (at 97.0788 44.0182) (layer B.SilkS)
     (effects (font (size 1.5 1.5) (thickness 0.25)) (justify mirror))
   )
-  (gr_text HOGALOG (at 93.7006 48.5394 90) (layer F.SilkS)
+  (gr_text HOG-A-LOG (at 93.7006 48.5394 90) (layer F.SilkS)
     (effects (font (size 3 1.6) (thickness 0.3)))
   )
