File: hog32a.kicad_pcb (KiCad board)
At the start: 2 copper layers, 51.6 x 75.9 mm, 38 parts, among them J1 REG:3V3, J10 Conn_01x07, J11 Conn_01x16, J12 dht22, J13 9602-a, J14 satx, J15 Conn_01x05, J16 LBO, J19 9602-b, J2 prog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

Commit message: update
Parts:
- Q1, Q2: value Q_NPN_CBE -> Q_NPN_EBC
- moved D1 3.53 mm to (101.9, 84.9)
- moved R8 3.36 mm to (105.2, 79.3)
- moved C6 2.45 mm to (108.0, 90.2)
- moved Q1 0.95 mm to (96.2, 70.2)
- moved Q2 0.77 mm to (96.3, 76.1)
- moved C5 0.70 mm to (109.8, 93.3)
- moved J3 0.40 mm to (98.4, 100.6)
Connections:
- Q1 pad 1: 0 -> DTR
- Q1 pad 3: DTR -> 0
- Q2 pad 1: RESET -> RTS
- Q2 pad 3: RTS -> RESET
Routing:
- net Net-(C1-Pad1): track 74.7 -> 66.9 mm
- net GND: track 324.1 -> 330.6 mm
- net RTS: track 28.2 -> 34.3 mm, vias 1 -> 0
- net 0: track 44.9 -> 49.7 mm, vias 1 -> 4
- net Net-(Q2-Pad2): track 17.3 -> 12.8 mm
- net RESET: track 89.4 -> 93.5 mm
- net 5:onewire: track 51.5 -> 53.9 mm
- net VBUS: track 7.43 -> 9.76 mm
- net VIN: track 85.5 -> 87.8 mm
- net DTR: track 34.4 -> 35.4 mm, vias 2 -> 1
- net +5V: track 92.7 -> 91.9 mm
Other:
- board text added: "+"
- board text added: "-"
- board text added: "0"
- board text added: "12"
- board text added: "13"
- board text added: "14"
- board text added: "15"
- board text added: "16"
- board text added: "17"
- board text added: "18"
- board text added: "19"
- board text added: "2"
- board text added: "21"
- board text added: "22"
- board text added: "23"
- board text added: "25"
- board text added: "26"
- board text added: "27"
- board text added: "32"
- board text added: "33"
- board text added: "34"
- board text added: "35"
- board text added: "3V3"
- board text added: "4"
- board text added: "5"
- board text added: "5V"
- board text added: "DIO5"
- board text added: "DTR"
- board text added: "GND"
- board text added: "QUAHOG-A-LOG"
- board text added: "RST"
- board text added: "RTS"
- board text added: "RX"
- board text added: "TX"
- board text added: "VBS"
- board text added: "VIN"
- board text added: "http://edgecollective.io/quahog-a-log"
- board text removed: "HOG-A-LOG"
- board text removed: "http://edgecollective.io/hog-a-log"

Commit message: update
Other:
- outline, holes or cut-outs redrawn
- board text added: "QUAHOG"
- board text added: "http://edgecollective.io/quahog"
- board text removed: "QUAHOG-A-LOG"
- board text removed: "http://edgecollective.io/quahog-a-log"
Changed lines of the file:
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@@
     (area 71.88881 27.94218 126.97242 108.04)
     (thickness 1.6)
-    (drawings 78)
+    (drawings 88)
     (tracks 816)
     (zones 0)
@@
     (descr "C, Disc series, Radial, pin pitch=2.50mm, , diameter*width=3.0*1.6mm^2, Capacitor, http://www.vishay.com/docs/45233/krseries.pdf")
     (tags "C Disc series Radial pin pitch 2.50mm  diameter 3.0mm width 1.6mm Capacitor")
-    (fp_text reference C1 (at 2.44856 1.94056 270) (layer F.SilkS)
+    (fp_text reference C1 (at -1.79832 -0.01524 360) (layer F.SilkS)
       (effects (font (size 1 1) (thickness 0.15)))
     )
@@
     (descr "C, Disc series, Radial, pin pitch=2.50mm, , diameter*width=3.0*1.6mm^2, Capacitor, http://www.vishay.com/docs/45233/krseries.pdf")
     (tags "C Disc series Radial pin pitch 2.50mm  diameter 3.0mm width 1.6mm Capacitor")
-    (fp_text reference C2 (at -2.25044 -0.13716) (layer F.SilkS)
+    (fp_text reference C2 (at 0.03048 -1.81356) (layer F.SilkS)
       (effects (font (size 1 1) (thickness 0.15)))
     )
@@
     (descr "Through hole straight pin header, 1x08, 2.54mm pitch, single row")
     (tags "Through hole pin header THT 1x08 2.54mm single row")
-    (fp_text reference J19 (at 3.00976 -1.9558 180) (layer F.SilkS)
+    (fp_text reference J19 (at -0.83072 20.9296 270) (layer F.SilkS)
       (effects (font (size 1 1) (thickness 0.15)))
     )
@@
     )
   )
+  (gr_text 2 (at 100.41128 58.00852) (layer F.SilkS)
+    (effects (font (size 0.8 0.8) (thickness 0.125)))
+  )
+  (gr_text 14 (at 97.78492 57.99836) (layer F.SilkS)
+    (effects (font (size 0.8 0.8) (thickness 0.125)))
+  )
+  (gr_text GND (at 95.26524 58.02884) (layer F.SilkS)
+    (effects (font (size 0.8 0.8) (thickness 0.125)))
+  )
+  (gr_text 3V3 (at 92.63888 58.01868) (layer F.SilkS)
+    (effects (font (size 0.8 0.8) (thickness 0.125)))
+  )
+  (gr_line (start 113.04524 97.00768) (end 113.04524 97.0026) (angle 90) (layer F.SilkS) (width 0.2))
+  (gr_line (start 109.99724 97.00768) (end 113.04524 97.00768) (angle 90) (layer F.SilkS) (width 0.2))
+  (gr_line (start 110.60684 81.32572) (end 110.60684 96.98736) (angle 90) (layer F.SilkS) (width 0.2))
+  (gr_line (start 112.81664 81.34604) (end 109.99724 81.34604) (angle 90) (layer F.SilkS) (width 0.2))
+  (gr_circle (center 120.14708 32.84728) (end 121.39676 33.71596) (layer Edge.Cuts) (width 0.15))
+  (gr_circle (center 76.6826 104.18064) (end 77.93228 105.04932) (layer Edge.Cuts) (width 0.15))
   (gr_text 27 (at 80.68564 53.68544) (layer F.SilkS)
     (effects (font (size 0.5 0.5) (thickness 0.125)))
@@
     (effects (font (size 0.8 0.8) (thickness 0.2)))
   )
-  (gr_text + (at 101.86416 105.79608) (layer F.SilkS)
-    (effects (font (size 0.8 0.8) (thickness 0.2)))
-  )
-  (gr_text - (at 98.3996 105.78592) (layer F.SilkS)
-    (effects (font (size 0.8 0.8) (thickness 0.2)))
+  (gr_text + (at 101.85908 105.50144) (layer F.SilkS)
+    (effects (font (size 1.2 1.2) (thickness 0.2)))
+  )
+  (gr_text - (at 98.49104 105.51668) (layer F.SilkS)
+    (effects (font (size 1.2 1.2) (thickness 0.2)))
   )
   (gr_text 15 (at 105.82148 92.57284) (layer F.SilkS)
@@
     (effects (font (size 0.8 0.8) (thickness 0.2)))
   )
-  (gr_text DTR (at 111.47552 79.91856 90) (layer F.SilkS)
-    (effects (font (size 0.8 0.8) (thickness 0.2)))
-  )
-  (gr_text RTS (at 111.53648 82.72272 90) (layer F.SilkS)
-    (effects (font (size 0.8 0.8) (thickness 0.2)))
-  )
-  (gr_text TX (at 111.57204 85.16112 90) (layer F.SilkS)
+  (gr_text DTR (at 111.57712 79.73568 90) (layer F.SilkS)
+    (effects (font (size 0.8 0.8) (thickness 0.2)))
+  )
+  (gr_text RTS (at 111.64824 82.92592 90) (layer F.SilkS)
+    (effects (font (size 0.8 0.8) (thickness 0.2)))
+  )
+  (gr_text TX (at 111.67872 85.1916 90) (layer F.SilkS)
     (effects (font (size 0.8 0.8) (thickness 0.2)))
   )
@@
     (effects (font (size 0.8 0.8) (thickness 0.2)))
   )
-  (gr_text "ver 0.1" (at 95.64116 38.97884 90) (layer F.SilkS)
+  (gr_text "ver 0.1" (at 95.64624 37.93236 90) (layer F.SilkS)
     (effects (font (size 1 0.8) (thickness 0.125)))
   )
-  (gr_text http://edgecollective.io/quahog-a-log (at 97.0788 44.0182) (layer B.SilkS)
+  (gr_text http://edgecollective.io/quahog (at 97.0788 44.0182) (layer B.SilkS)
     (effects (font (size 1.5 1.5) (thickness 0.25)) (justify mirror))
   )
-  (gr_text QUAHOG-A-LOG (at 93.7006 48.5394 90) (layer F.SilkS)
-    (effects (font (size 2.8 1.5) (thickness 0.3)))
+  (gr_text QUAHOG (at 93.71076 47.72152 90) (layer F.SilkS)
+    (effects (font (size 2.8 3) (thickness 0.3)))
   )
   (gr_line (start 92.5576 100.0252) (end 106.0196 100.0252) (angle 90) (layer Dwgs.User) (width 0.2))
@@
   (segment (start 110.49 95.845) (end 110.5046 95.845) (width 0.35) (layer B.Cu) (net 3))
   (segment (start 108.82408 97.51092) (end 109.22032 97.51092) (width 0.35) (layer B.Cu) (net 3))
-  (segment (start 101.76256 96.5708) (end 100.965 95.25) (width 0.35) (layer B.Cu) (net 3) (status 800000))
+  (segment (start 101.76256 96.5708) (end 100.965 95.25) (width 0.35) (layer B.Cu) (net 3))
   (segment (start 102.54996 97.6376) (end 103.124 97.59696) (width 0.35) (layer B.Cu) (net 3))
   (segment (start 103.124 97.59696) (end 108.73804 97.59696) (width 0.35) (layer B.Cu) (net 3))
@@
   (segment (start 119.5578 46.8376) (end 116.3326 46.8376) (width 0.25) (layer F.Cu) (net 37))
   (segment (start 116.3326 46.8376) (end 116.315 46.82) (width 0.25) (layer F.Cu) (net 37))
-  (segment (start 92.51188 100.05568) (end 92.964 100.05568) (width 0.35) (layer F.Cu) (net 38) (status C00000))
-  (segment (start 92.964 100.05568) (end 95.01632 98.00336) (width 0.35) (layer F.Cu) (net 38) (status 400000))
-  (segment (start 112.6998 101.81844) (end 112.6998 100.0506) (width 0.35) (layer B.Cu) (net 38) (status 800000))
+  (segment (start 92.51188 100.05568) (end 92.964 100.05568) (width 0.35) (layer F.Cu) (net 38))
+  (segment (start 92.964 100.05568) (end 95.01632 98.00336) (width 0.35) (layer F.Cu) (net 38))
+  (segment (start 112.6998 101.81844) (end 112.6998 100.0506) (width 0.35) (layer B.Cu) (net 38))
   (segment (start 111.63808 102.88016) (end 112.6998 101.81844) (width 0.35) (layer B.Cu) (net 38))
   (segment (start 106.49712 102.88016) (end 111.63808 102.88016) (width 0.35) (layer B.Cu) (net 38))
