File: hog32a.sch (KiCad schematic (older format))
At the start: 39 parts, among them J1 REG:3V3, J10 Conn_01x07, J11 Conn_01x16, J12 dht22, J13 9602-a, J14 satx, J15 Conn_01x05, J16 LBO, J19 9602-b, J2 prog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

Commit message: update
Connections:
- net 18:dht22 is gone; now on net 18:DHT22: J12.2 (Pin_2), R7.2, U1.30 (IO18)
- no-connect marks 6 -> 15
Changed lines of the file:
@@
 19
 Text GLabel 6600 2350 2    60   Input ~ 0
-18:dht22
+18:DHT22
 Text GLabel 6600 2450 2    60   Input ~ 0
 5:onewire
@@
 15
 Text GLabel 5250 4750 0    60   Input ~ 0
-18:dht22
+18:DHT22
 $Comp
 L GND #PWR035
@@
 Text Notes 1100 4250 0    60   ~ 0
 Manual Reset
+NoConn ~ 10250 1450
+NoConn ~ 5450 3450
+NoConn ~ 5550 3450
+NoConn ~ 5650 3450
+NoConn ~ 5750 3450
+NoConn ~ 5850 3450
+NoConn ~ 5950 3450
+NoConn ~ 5850 4650
+NoConn ~ 3350 2800
 $EndSCHEMATC

Commit message: update
Parts:
- removed J8: Conn_01x01, SMD_Packages:1Pin, symbol Conn_01x01
Changed lines of the file:
@@
 NoConn ~ 4750 2000
 NoConn ~ 4750 2100
-$Comp
-L Conn_01x01 J8
-U 1 1 5BAB5619
-P 6900 2950
-F 0 "J8" H 6900 3050 50  0000 C CNN
-F 1 "Conn_01x01" H 6900 2850 50  0000 C CNN
-F 2 "SMD_Packages:1Pin" H 6900 2950 50  0001 C CNN
-F 3 "" H 6900 2950 50  0001 C CNN
-	1    6900 2950
-	1    0    0    -1
-$EndComp
 NoConn ~ 6600 2150
 $Comp
@@
 Connection ~ 1350 1900
 Connection ~ 1350 2500
-Wire Wire Line
-	6600 2950 6700 2950
 Wire Wire Line
 	6700 2950 6700 3150
@@
 NoConn ~ 5850 4650
 NoConn ~ 3350 2800
+Connection ~ 6700 2950
+Wire Wire Line
+	6600 2950 6700 2950
 $EndSCHEMATC

Commit message: update
Parts:
- removed Q1, Q2: Q_NPN_CBE, TO_SOT_Packages_THT:TO-92_Molded_Narrow, symbol Q_NPN_CBE
- added Q1, Q2: Q_NPN_EBC, symbol Q_NPN_EBC
Connections:
- net 0: now also Q1.3 (C)
- net DTR: now also Q1.1 (E)
- net RESET: now also Q2.3 (C)
- net RTS: now also Q2.1 (E)
- net at R2.1: now also Q1.2 (B)
- net at R3.1: now also Q2.2 (B)
Changed lines of the file:
@@
-$EndComp
-$Comp
-L Q_NPN_CBE Q2
-U 1 1 5B888A61
-P 3600 5550
-F 0 "Q2" H 3800 5600 50  0000 L CNN
-F 1 "Q_NPN_CBE" H 3800 5500 50  0000 L CNN
-F 2 "TO_SOT_Packages_THT:TO-92_Molded_Narrow" H 3800 5650 50  0001 C CNN
-F 3 "" H 3600 5550 50  0001 C CNN
-	1    3600 5550
-	1    0    0    1
 $EndComp
 $Comp
@@
 Text GLabel 8550 2250 0    60   Input ~ 0
 5:onewire
-$Comp
-L Q_NPN_CBE Q1
-U 1 1 5B8887FC
-P 3600 4950
-F 0 "Q1" H 3800 5000 50  0000 L CNN
-F 1 "Q_NPN_CBE" H 3800 4900 50  0000 L CNN
-F 2 "TO_SOT_Packages_THT:TO-92_Molded_Narrow" H 3800 5050 50  0001 C CNN
-F 3 "" H 3600 4950 50  0001 C CNN
-	1    3600 4950
-	1    0    0    -1
-$EndComp
 NoConn ~ 4750 2000
 NoConn ~ 4750 2100
@@
 Wire Wire Line
 	6600 2950 6700 2950
+$Comp
+L Q_NPN_EBC Q1
+U 1 1 5BABD1AE
+P 3600 4950
+F 0 "Q1" H 3800 5000 50  0000 L CNN
+F 1 "Q_NPN_EBC" H 3800 4900 50  0000 L CNN
+F 2 "" H 3800 5050 50  0001 C CNN
+F 3 "" H 3600 4950 50  0001 C CNN
+	1    3600 4950
+	1    0    0    -1
+$EndComp
+$Comp
+L Q_NPN_EBC Q2
+U 1 1 5BABD59D
+P 3600 5550
+F 0 "Q2" H 3800 5600 50  0000 L CNN
+F 1 "Q_NPN_EBC" H 3800 5500 50  0000 L CNN
+F 2 "" H 3800 5650 50  0001 C CNN
+F 3 "" H 3600 5550 50  0001 C CNN
+	1    3600 5550
+	1    0    0    1
+$EndComp
 $EndSCHEMATC
